File: demo project.kicad_sch (KiCad schematic)
At the start: 37 parts, among them J1 Conn_ARM_SWD_TagConnect_TC2030, J2 USB_C_Receptacle_USB2.0_16P, U1 MSPM0G3507SPTR, U2 USBLC6-2SC6, U3 LIS2DH, U4 SPX3819M5-L-3-3, U5 CH340E, X1 8MHz

Commit message: added some netclasses with some colors
Connections:
- net GND: now also U5.3 (GND)
- net SWDIO: now reaches J1.2 (SWDIO), U1.34 (PA19/SWDIO)
- net SWCLK: now reaches J1.4 (SWCLK), U1.35 (PA20/SWCLK)
- net SCL renamed I2C_SCL
- net SDA renamed I2C_SDA
Changed lines of the file:
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@@
 	)
 	(junction
+		(at 193.04 134.62)
+		(diameter 0)
+		(color 0 0 0 0)
+	)
+	(junction
 		(at 224.79 105.41)
 		(diameter 0)
@@
 	(wire
 		(pts
+			(xy 254 93.98) (xy 254 96.52)
+		)
+		(stroke
+			(width 0)
+			(type default)
+		)
+	)
+	(wire
+		(pts
 			(xy 264.16 88.9) (xy 278.13 88.9)
 		)
@@
 	(wire
 		(pts
-			(xy 193.04 121.92) (xy 193.04 138.43)
+			(xy 193.04 121.92) (xy 193.04 134.62)
 		)
 		(stroke
@@
 	(wire
 		(pts
+			(xy 193.04 134.62) (xy 193.04 138.43)
+		)
+		(stroke
+			(width 0)
+			(type default)
+		)
+	)
+	(wire
+		(pts
 			(xy 49.53 53.34) (xy 64.77 53.34)
 		)
@@
 		)
 	)
+	(label "SWCLK"
+		(at 118.11 80.01 0)
+		(effects
+			(font
+				(size 1.27 1.27)
+			)
+			(justify left bottom)
+		)
+	)
 	(label "HFXIN"
 		(at 46.99 85.09 0)
@@
 		)
 	)
-	(label "SCL"
+	(label "I2C_SCL"
 		(at 184.15 124.46 0)
 		(effects
@@
 		)
 	)
-	(label "SDA"
+	(label "I2C_SDA"
 		(at 55.88 93.98 0)
 		(effects
@@
 		)
 	)
-	(label "SDA"
+	(label "I2C_SDA"
 		(at 184.15 119.38 0)
 		(effects
@@
 		)
 	)
+	(label "SWDIO"
+		(at 118.11 77.47 0)
+		(effects
+			(font
+				(size 1.27 1.27)
+			)
+			(justify left bottom)
+		)
+	)
 	(label "INT1"
 		(at 219.71 119.38 0)
@@
 		)
 	)
-	(label "SCL"
+	(label "I2C_SCL"
 		(at 55.88 91.44 0)
 		(effects
@@
 	)
 	(symbol
+		(lib_id "power:PWR_FLAG")
+		(at 193.04 134.62 90)
+		(unit 1)
+		(body_style 1)
+		(exclude_from_sim no)
+		(in_bom yes)
+		(on_board yes)
+		(in_pos_files yes)
+		(dnp no)
+		(fields_autoplaced yes)
+		(property "Reference" "#FLG07"
+			(at 191.135 134.62 0)
+			(hide yes)
+			(show_name no)
+			(do_not_autoplace no)
+			(effects
+				(font
+					(size 1.27 1.27)
+				)
+			)
+		)
+		(property "Value" "PWR_FLAG"
+			(at 189.23 134.6199 90)
+			(show_name no)
+			(do_not_autoplace no)
+			(effects
+				(font
+					(size 1.27 1.27)
+				)
+				(justify left)
+			)
+		)
+		(property "Footprint" ""
+			(at 193.04 134.62 0)
+			(hide yes)
+			(show_name no)
+			(do_not_autoplace no)
+			(effects
+				(font
+					(size 1.27 1.27)
+				)
+			)
+		)
+		(property "Datasheet" ""
+			(at 193.04 134.62 0)
+			(hide yes)
+			(show_name no)
+			(do_not_autoplace no)
+			(effects
+				(font
+					(size 1.27 1.27)
+				)
+			)
+		)
+		(property "Description" "Special symbol for telling ERC where power comes from"
+			(at 193.04 134.62 0)
+			(hide yes)
+			(show_name no)
+			(do_not_autoplace no)
+			(effects
+				(font
+					(size 1.27 1.27)
+				)
+			)
+		)
+		(pin "1"
+		)
+		(instances
+			(project "demo project"
+				(path "/fec0df47-5383-43eb-b5c3-4e96b04be4f5"
+					(reference "#FLG07")
+					(unit 1)
+				)
+			)
+		)
+	)
+	(symbol
 		(lib_id "power:GND")
 		(at 205.74 137.16 0)
@@
 					(unit 1)
 				)
+			)
+		)
+	)
+	(symbol
+		(lib_id "power:GND")
+		(at 254 96.52 0)
+		(unit 1)
+		(body_style 1)
+		(exclude_from_sim no)
+		(in_bom yes)
+		(on_board yes)
+		(in_pos_files yes)
+		(dnp no)
+		(fields_autoplaced yes)
+		(property "Reference" "#PWR035"
+			(at 254 102.87 0)
+			(hide yes)
+			(show_name no)
+			(do_not_autoplace no)
+			(effects
+				(font
+					(size 1.27 1.27)
+				)
+			)
+		)
+		(property "Value" "GND"
+			(at 254 101.6 0)
+			(show_name no)
+			(do_not_autoplace no)
+			(effects
+				(font
+					(size 1.27 1.27)
+				)
+			)
+		)
+		(property "Footprint" ""
+			(at 254 96.52 0)
+			(hide yes)
+			(show_name no)
+			(do_not_autoplace no)
+			(effects
+				(font
+					(size 1.27 1.27)
+				)
+			)
+		)
+		(property "Datasheet" ""
+			(at 254 96.52 0)
+			(hide yes)
+			(show_name no)
+			(do_not_autoplace no)
+			(effects
+				(font
+					(size 1.27 1.27)
+				)
+			)
+		)
+		(property "Description" "Power symbol creates a global label with name \"GND\" , ground"
+			(at 254 96.52 0)
+			(hide yes)
+			(show_name no)
+			(do_not_autoplace no)
+			(effects
+				(font
+					(size 1.27 1.27)
+				)
+			)
+		)
+		(pin "1"
+		)
+		(instances
+			(project "demo project"
+				(path "/fec0df47-5383-43eb-b5c3-4e96b04be4f5"
+					(reference "#PWR035")
+					(unit 1)
+				)

Commit message: Placement and routing
Connections:
- net I2C_SCL: now also U1.19 (PA11); no longer U1.14 (PB2)
- net I2C_SDA: now also U1.18 (PA10/CLK_OUT); no longer U1.15 (PB3)
Changed lines of the file:
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@@
 	)
 	(no_connect
+		(at 64.77 91.44)
+	)
+	(no_connect
 		(at 110.49 109.22)
 	)
@@
 	)
 	(no_connect
-		(at 64.77 104.14)
-	)
-	(no_connect
 		(at 64.77 78.74)
 	)
@@
 	)
 	(no_connect
-		(at 64.77 81.28)
+		(at 64.77 93.98)
 	)
 	(no_connect
-		(at 64.77 101.6)
+		(at 64.77 81.28)
 	)
 	(no_connect
@@
 	(wire
 		(pts
-			(xy 53.34 91.44) (xy 64.77 91.44)
-		)
-		(stroke
-			(width 0)
-			(type default)
-		)
-	)
-	(wire
-		(pts
 			(xy 100.33 26.67) (xy 100.33 27.94)
 		)
@@
 	(wire
 		(pts
+			(xy 54.61 104.14) (xy 64.77 104.14)
+		)
+		(stroke
+			(width 0)
+			(type default)
+		)
+	)
+	(wire
+		(pts
 			(xy 118.11 86.36) (xy 118.11 80.01)
 		)
@@
 	(wire
 		(pts
+			(xy 54.61 101.6) (xy 64.77 101.6)
+		)
+		(stroke
+			(width 0)
+			(type default)
+		)
+	)
+	(wire
+		(pts
 			(xy 83.82 33.02) (xy 83.82 48.26)
 		)
@@
 	(wire
 		(pts
-			(xy 53.34 93.98) (xy 64.77 93.98)
-		)
-		(stroke
-			(width 0)
-			(type default)
-		)
-	)
-	(wire
-		(pts
 			(xy 144.78 90.17) (xy 149.86 90.17)
 		)
@@
 	(wire
 		(pts
-			(xy 170.18 69.85) (xy 170.18 72.39)
+			(xy 170.18 69.85) (xy 170.18 74.93)
 		)
 		(stroke
@@
 	(wire
 		(pts
-			(xy 162.56 69.85) (xy 162.56 72.39)
+			(xy 162.56 69.85) (xy 162.56 73.66)
 		)
 		(stroke
@@
 		)
 	)
+	(label "I2C_SCL"
+		(at 55.88 104.14 0)
+		(effects
+			(font
+				(size 1.27 1.27)
+			)
+			(justify left bottom)
+		)
+	)
 	(label "SWCLK"
 		(at 118.11 80.01 0)
@@
 		)
 	)
+	(label "I2C_SDA"
+		(at 55.88 101.6 0)
+		(effects
+			(font
+				(size 1.27 1.27)
+			)
+			(justify left bottom)
+		)
+	)
 	(label "I2C_SCL"
 		(at 184.15 124.46 0)
@@
 		)
 	)
-	(label "I2C_SDA"
-		(at 55.88 93.98 0)
-		(effects
-			(font
-				(size 1.27 1.27)
-			)
-			(justify left bottom)
-		)
-	)
 	(label "VREF-"
 		(at 115.57 96.52 0)
@@
 		)
 	)
-	(label "I2C_SCL"
-		(at 55.88 91.44 0)
-		(effects
-			(font
-				(size 1.27 1.27)
-			)
-			(justify left bottom)
-		)
-	)
 	(label "HFXOUT"
 		(at 46.99 87.63 0)
@@
 	(symbol
 		(lib_id "power:GND")
-		(at 162.56 72.39 0)
+		(at 162.56 73.66 0)
 		(unit 1)
 		(body_style 1)
@@
 		(fields_autoplaced yes)
 		(property "Reference" "#PWR013"
-			(at 162.56 78.74 0)
+			(at 162.56 80.01 0)
 			(hide yes)
 			(show_name no)
@@
 		)
 		(property "Value" "GND"
-			(at 162.56 77.47 0)
+			(at 162.56 78.74 0)
 			(show_name no)
 			(do_not_autoplace no)
@@
 		)
 		(property "Footprint" ""
-			(at 162.56 72.39 0)
+			(at 162.56 73.66 0)
 			(hide yes)
 			(show_name no)
@@
 		)
 		(property "Datasheet" ""
-			(at 162.56 72.39 0)
+			(at 162.56 73.66 0)
 			(hide yes)
 			(show_name no)
@@
 		)
 		(property "Description" "Power symbol creates a global label with name \"GND\" , ground"
-			(at 162.56 72.39 0)
+			(at 162.56 73.66 0)
 			(hide yes)
 			(show_name no)
@@
 	(symbol
 		(lib_id "power:GND")
-		(at 170.18 72.39 0)
+		(at 170.18 74.93 0)
 		(unit 1)
 		(body_style 1)
@@
 		(fields_autoplaced yes)
 		(property "Reference" "#PWR014"
-			(at 170.18 78.74 0)
+			(at 170.18 81.28 0)
 			(hide yes)
 			(show_name no)
@@
 		)
 		(property "Value" "GND"
-			(at 170.18 77.47 0)
+			(at 170.18 80.01 0)
 			(show_name no)
 			(do_not_autoplace no)
@@
 		)
 		(property "Footprint" ""
-			(at 170.18 72.39 0)
+			(at 170.18 74.93 0)
 			(hide yes)
 			(show_name no)
@@
 		)
 		(property "Datasheet" ""
-			(at 170.18 72.39 0)
+			(at 170.18 74.93 0)
 			(hide yes)
 			(show_name no)
@@
 		)
 		(property "Description" "Power symbol creates a global label with name \"GND\" , ground"
-			(at 170.18 72.39 0)
+			(at 170.18 74.93 0)
 			(hide yes)
 			(show_name no)
