File: demo project.kicad_pcb (KiCad board)
At the start: 2 copper layers, 37 parts, among them J1 Conn_ARM_SWD_TagConnect_TC2030, J2 USB_C_Receptacle_USB2.0_16P, U1 MSPM0G3507SPTR, U2 USBLC6-2SC6, U3 LIS2DH, U4 SPX3819M5-L-3-3, U5 CH340E, X1 8MHz

Commit message: Placement and routing
Parts:
- moved FID2 106.0 mm to (122.5, 115.5)
- moved FID3 104.0 mm to (122.5, 94.8)
- moved U2 96.7 mm to (124.0, 105.2)
- moved R6 91.2 mm to (121.5, 111.5)
- moved U4 91.0 mm to (132.4, 96.5)
- moved J2 90.8 mm to (116.5, 105.0), turned to -90 degrees
- moved R7 90.3 mm to (121.0, 98.5)
- moved C11 88.3 mm to (128.9, 96.5), turned to -90 degrees
- moved X1 87.4 mm to (137.9, 111.7)
- moved R8 86.6 mm to (124.8, 102.2)
- moved C14 82.2 mm to (135.9, 96.5), turned to -90 degrees
- moved C1 80.7 mm to (134.7, 111.7), turned to 90 degrees
- moved MH4 80.3 mm to (117.0, 115.0)
- moved MH1 80.3 mm to (117.0, 95.0)
- moved C7 79.3 mm to (124.0, 100.0), turned to 90 degrees
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Connections:
- U1 pad 14: /I2C_SCL -> unconnected-(U1-PB2-Pad14)
- U1 pad 15: /I2C_SDA -> unconnected-(U1-PB3-Pad15)
- U1 pad 18: unconnected-(U1-PA10/CLK_OUT-Pad18) -> /I2C_SDA
- U1 pad 19: unconnected-(U1-PA11-Pad19) -> /I2C_SCL
Routing:
- net +3V3: track 0.00 -> 90.2 mm, vias 0 -> 7
- net /UART0CTS: track 0.00 -> 36.4 mm
- net /UART0RTS: track 0.00 -> 33.9 mm
- net /NRST: track 0.00 -> 25.2 mm
- net /INT2: track 0.00 -> 17.8 mm
- net +VBUS: track 0.00 -> 17.7 mm, vias 0 -> 2
- net /HFXIN: track 0.00 -> 17.7 mm
- net GND: track 0.00 -> 17.1 mm, vias 0 -> 136
- net /INT1: track 0.00 -> 16.1 mm
- net /SWCLK: track 0.00 -> 15.5 mm
- net +VBUSF: track 0.00 -> 14.4 mm
- net /USBD-: track 0.00 -> 10.9 mm
- net /SWDIO: track 0.00 -> 10.5 mm
- net /UART_TX: track 0.00 -> 9.55 mm
- net /UART_RX: track 0.00 -> 9.55 mm
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- added copper zone on B.Cu, net GND
- added copper zone on F.Cu, net GND
Other:
- board outline added: 53.5 x 28.5 mm

Commit message: Unsaved changes on pcb and schematics page
Other:
- board text added: "DEMO PCB"
Changed lines of the file:
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@@
 		(grid_origin 112.5 119.5)
 		(pcbplotparams
-			(layerselection 0x00000000_00000000_55555555_5755f5ff)
+			(layerselection 0x00000000_00000000_55555555_5755757f)
 			(plot_on_all_layers_selection 0x00000000_00000000_00000000_00000000)
 			(disableapertmacros no)
@@
 			(usegerberattributes yes)
 			(usegerberadvancedattributes yes)
-			(creategerberjobfile yes)
+			(creategerberjobfile no)
 			(dashed_line_dash_ratio 12)
 			(dashed_line_gap_ratio 3)
@@
 			(plotframeref no)
 			(mode 1)
-			(useauxorigin no)
+			(useauxorigin yes)
 			(pdf_front_fp_property_popups yes)
 			(pdf_back_fp_property_popups yes)
@@
 			(plotpadnumbers no)
 			(hidednponfab no)
-			(sketchdnponfab yes)
-			(crossoutdnponfab yes)
+			(sketchdnponfab no)
+			(crossoutdnponfab no)
 			(subtractmaskfromsilk no)
 			(outputformat 1)
 			(mirror no)
-			(drillshape 1)
+			(drillshape 0)
 			(scaleselection 1)
-			(outputdirectory "")
+			(outputdirectory "manufacturing/")
 		)
 	)
@@
 			(net "GND")
 			(pintype "passive")
+			(zone_connect 2)
 		)
 		(embedded_fonts no)
@@
 		(sheetname "/")
 		(sheetfile "demo project.kicad_sch")
-		(units
-			(unit
-				(name "A")
-				(pins "S1" "B1" "B12" "A1" "A12" "A9" "B4" "B9" "A4" "A7" "B7" "A6" "B6"
-					"A5" "B5" "A8" "B8"
-				)
-			)
-		)
 		(attr smd)
 		(duplicate_pad_numbers_are_jumpers no)
@@
 		)
 		(pad "A1" smd roundrect
-			(at -3.2 -3.68 270)
+			(at -3.2 -3.8 270)
 			(size 0.6 1.15)
 			(layers "F.Cu" "F.Mask" "F.Paste")
@@
 			(pinfunction "GND_A1")
 			(pintype "passive")
+			(zone_connect 2)
 		)
 		(pad "A4" smd roundrect
-			(at -2.4 -3.68 270)
+			(at -2.4 -3.755 270)
 			(size 0.6 1.15)
 			(layers "F.Cu" "F.Mask" "F.Paste")
@@
 		)
 		(pad "A9" smd roundrect
-			(at 2.4 -3.68 270)
+			(at 2.4 -3.8 270)
 			(size 0.6 1.15)
 			(layers "F.Cu" "F.Mask" "F.Paste")
@@
 		)
 		(pad "A12" smd roundrect
-			(at 3.2 -3.68 270)
+			(at 3.2 -3.8 270)
 			(size 0.6 1.15)
 			(layers "F.Cu" "F.Mask" "F.Paste")
@@
 			(pinfunction "GND_A12")
 			(pintype "passive")
+			(zone_connect 2)
 		)
 		(pad "B1" smd roundrect
-			(at 3.2 -3.68 270)
+			(at 3.2 -3.8 270)
 			(size 0.6 1.15)
 			(layers "F.Cu" "F.Mask" "F.Paste")
@@
 			(pinfunction "GND_B1")
 			(pintype "passive")
+			(zone_connect 2)
 		)
 		(pad "B4" smd roundrect
-			(at 2.4 -3.68 270)
+			(at 2.4 -3.8 270)
 			(size 0.6 1.15)
 			(layers "F.Cu" "F.Mask" "F.Paste")
@@
 		)
 		(pad "B9" smd roundrect
-			(at -2.4 -3.68 270)
+			(at -2.4 -3.755 270)
 			(size 0.6 1.15)
 			(layers "F.Cu" "F.Mask" "F.Paste")
@@
 		)
 		(pad "B12" smd roundrect
-			(at -3.2 -3.68 270)
+			(at -3.2 -3.8 270)
 			(size 0.6 1.15)
 			(layers "F.Cu" "F.Mask" "F.Paste")
@@
 			(pinfunction "GND_B12")
 			(pintype "passive")
+			(zone_connect 2)
 		)
 		(pad "SH" thru_hole oval
@@
 			(pinfunction "GND_5")
 			(pintype "power_in")
+			(zone_connect 2)
 		)
 		(pad "6" connect circle
@@
 		(layer "Edge.Cuts")
 	)
+	(gr_text "DEMO PCB"
+		(at 134.75 93.75 0)
+		(layer "F.SilkS")
+		(effects
+			(font
+				(size 1.5 1.5)
+				(thickness 0.3)
+				(bold yes)
+			)
+			(justify left bottom)
+		)
+	)
 	(segment
 		(start 140.75 108.25)
@@
 	)
 	(segment
-		(start 147.963447 115.039254)
-		(end 147.961693 115.0375)
-		(width 0.2)
-		(layer "F.Cu")
-		(net "+3V3")
-	)
-	(segment
 		(start 139.431704 103.618296)
 		(end 139.25 103.8)
@@
 	)
 	(segment
+		(start 148.211693 115.2875)
+		(end 148.75 115.2875)
+		(width 0.3)
+		(layer "F.Cu")
+		(net "+3V3")
+	)
+	(segment
 		(start 149.7125 115.2875)
 		(end 149.75 115.25)
@@
 	)
 	(segment
-		(start 147.5125 115.0375)
-		(end 147.961693 115.0375)
-		(width 0.152)
-		(layer "F.Cu")
-		(net "+3V3")
-	)
-	(segment
-		(start 148.5 115.0375)
-		(end 148.75 115.2875)
-		(width 0.3)
-		(layer "F.Cu")
-		(net "+3V3")
-	)
-	(segment
 		(start 141 115.5)
 		(end 141.5 115)
@@
 	)
 	(segment
+		(start 147.961693 115.0375)
+		(end 148.211693 115.2875)
+		(width 0.3)
+		(layer "F.Cu")
+		(net "+3V3")
+	)
+	(segment
 		(start 145.63831 115)
 		(end 145.72781 115.0895)
@@
 	)
 	(segment
-		(start 147.961693 115.0375)
-		(end 148.5 115.0375)
-		(width 0.3)
+		(start 147.5125 115.0375)
+		(end 147.961693 115.0375)
+		(width 0.152)
 		(layer "F.Cu")
 		(net "+3V3")
